Commit message: update

File: cocoax/src/cocoax_description/description/cocoax_robot_core.xacro (robot description, xacro)
@@ -31,5 +31,5 @@
     </link>
     <!-- LEFT WHEEL LINK -->
-    <joint name="left_wheel_joint" type="continuous">
+    <joint name="left_wheel_joint" type="fixed"> <!-- continuous -->
         <parent link="base_link"/>
         <child link="left_wheel"/>
@@ -54,5 +54,5 @@
     </link>
     <!-- RIGHT WHEEL LINK -->
-    <joint name="right_wheel_joint" type="continuous">
+    <joint name="right_wheel_joint" type="fixed">
         <parent link="base_link"/>
         <child link="right_wheel"/>
