Commit message: update

File: cocoam/src/cocoam_description/description/cocoam_robot.urdf.xacro (robot description, xacro)
@@ -2,3 +2,4 @@
 <robot xmlns:xacro="http://www.ros.org/wiki/xacro"  name="robot">
     <xacro:include filename="cocoam_robot_core.xacro" />
+    <xacro:include filename="gazebo_control.xacro" />
 </robot>

File: cocoam/src/cocoam_description/description/cocoam_robot_core.xacro (robot description, xacro)
@@ -31,5 +31,5 @@
     </link>
     <!-- LEFT WHEEL LINK -->
-    <joint name="left_wheel_joint" type="fixed"> <!-- continuous -->
+    <joint name="left_wheel_joint" type="continuous"> <!-- continuous -->
         <parent link="base_link"/>
         <child link="left_wheel"/>
@@ -53,6 +53,9 @@
         </xacro:inertial_cylinder>
     </link>
+    <gazebo reference="left_wheel">
+        <material>Gazebo/Blue</material>
+    </gazebo>
     <!-- RIGHT WHEEL LINK -->
-    <joint name="right_wheel_joint" type="fixed">
+    <joint name="right_wheel_joint" type="continuous"> <!-- continuous -->
         <parent link="base_link"/>
         <child link="right_wheel"/>
@@ -76,4 +79,7 @@
         </xacro:inertial_cylinder>
     </link>
+    <gazebo reference="right_wheel">
+        <material>Gazebo/Blue</material>
+    </gazebo>
     <!-- CASTER WHEEL LINK -->
     <joint name="caster_wheel_joint" type="fixed">
@@ -98,3 +104,8 @@
         </xacro:inertial_sphere>
     </link>
+    <gazebo reference="caster_wheel">
+        <material>Gazebo/Black</material>
+        <mu1 value="0.001"/>
+        <mu2 value="0.001"/>
+    </gazebo>
 </robot>
