Commit message: update

File: cocoam/src/cocoam_description/description/cocoam_include.xacro (robot description, xacro)
@@ -3,23 +3,23 @@
     <!-- This file is not a robot in and of itself, it just contains some useful tags that could be included in any robot -->
     <!-- add more codes -->
-    <material name="Grey">
+    <material name="grey">
         <color rgba="0.2 0.2 0.2 1.0"/>
     </material>
-    <material name="Orange">
+    <material name="orange">
         <color rgba="1.0 0.423529411765 0.0392156862745 1.0"/>
     </material>
-    <material name="Blue">
+    <material name="blue">
         <color rgba="0.0 0.5 1.0 1.0"/>
     </material>
-    <material name="Red">
+    <material name="red">
     <color rgba="1.0 0.0 0.0 1.0"/>
     </material>
-    <material name="Black">
+    <material name="black">
         <color rgba="0.0 0.0 0.0 0.6"/>
     </material>
-    <material name="White">
+    <material name="white">
         <color rgba="1.0 1.0 1.0 1.0"/>
     </material>
-    <material name="DarkBlue">
+    <material name="darkblue">
         <color rgba="0.0 0.0 0.3764 0.6"/>
     </material>

File: cocoam/src/cocoam_description/description/cocoam_robot_core.xacro (robot description, xacro)
@@ -18,5 +18,5 @@
                 <box size="0.3 0.3 0.15"/>
             </geometry>
-            <material name="White"/>
+            <material name="white"/>
         </visual>
         <collision>
@@ -42,5 +42,5 @@
                 <cylinder radius="0.05" length="0.04"/>
             </geometry>
-            <material name="Blue"/>
+            <material name="blue"/>
         </visual>
         <collision>
@@ -65,5 +65,5 @@
                 <cylinder radius="0.05" length="0.04"/>
             </geometry>
-            <material name="Blue"/>
+            <material name="blue"/>
         </visual>
         <collision>
@@ -87,5 +87,5 @@
                 <sphere radius="0.05"/>
             </geometry>
-            <material name="Black"/>
+            <material name="black"/>
         </visual>
         <collision>

Commit message: zhbbot

File: cocoam/src/cocoam_description/description/cocoam_include.xacro (robot description, xacro)
@@ -13,5 +13,5 @@
     </material>
     <material name="red">
-    <color rgba="1.0 0.0 0.0 1.0"/>
+        <color rgba="1.0 0.0 0.0 1.0"/>
     </material>
     <material name="black">

File: cocoam/src/cocoam_description/description/cocoam_robot.urdf.xacro (robot description, xacro)
@@ -5,3 +5,12 @@
     <xacro:include filename="cocoam_ros2_control.xacro" />
     <xacro:include filename="lidar.xacro" />
+<!--
+    <xacro:arg name="use_ros2_control" default="true"/>
+    <xacro:include filename="cocoam_robot_core.xacro"/>
+    <xacro:if value="$(arg use_ros2_control)">
+        <xacro:include filename="cocoam_ros2_control.xacro" />
+    </xacro:if>
+    <xacro:unless value="$(arg use_ros2_control)">
+        <xacro:include filename="gazebo_control.xacro" />
+    </xacro:unless> -->
 </robot>

File: cocoam/src/cocoam_description/description/cocoam_robot_core.xacro (robot description, xacro)
@@ -5,4 +5,12 @@
     <!-- BASE LINK -->
     <link name="base_link">
+    </link>
+    <!-- BASE_FOOTPRINT LINK -->
+    <joint name="base_footprint_joint" type="fixed">
+        <parent link="base_link"/>
+        <child link="base_footprint"/>
+        <origin xyz="0 0 0" rpy="0 0 0"/>
+    </joint>
+    <link name="base_footprint">
     </link>
     <!-- CHASSIS LINK -->
@@ -26,5 +34,5 @@
             </geometry>
         </collision>
-        <xacro:inertial_box mass="0.5" x="0.3" y="0.3" z="0.15">
+        <xacro:inertial_box mass="1.5" x="0.3" y="0.3" z="0.15">
             <origin xyz="0.15 0 0.075" rpy="0 0 0"/>
         </xacro:inertial_box>
@@ -100,5 +108,5 @@
             </geometry>
         </collision>
-        <xacro:inertial_sphere mass="0.1" radius="0.05">
+        <xacro:inertial_sphere mass="0.5" radius="0.05">
             <origin xyz="0 0 0" rpy="0 0 0"/>
         </xacro:inertial_sphere>

File: zhbbot/src/zhbbot_description/description/zhbbot_addon.xacro (robot description, xacro)
@@ -1,8 +1,9 @@
 <?xml version="1.0"?>
 <robot xmlns:xacro="http://www.ros.org/wiki/xacro" >
+    <!-- Laser  -->
     <joint name="laser_joint" type="fixed">
-        <parent link="chassis"/>
+        <parent link="base_link"/>
         <child link="laser_frame"/>
-        <origin xyz="0.1 0 0.175" rpy="0 0 0"/>
+        <origin xyz="0.122 0 0.312" rpy="0 0 0"/>
     </joint>
     <link name="laser_frame">
@@ -10,4 +11,11 @@
             <geometry>
                 <cylinder radius="0.05" length="0.04"/>
+            </geometry>
+            <material name="red"/>
+        </visual>
+        <visual>
+            <origin xyz="0 0 -0.05"/>
+            <geometry>
+                <cylinder radius="0.01" length="0.1"/>
             </geometry>
             <material name="red"/>
@@ -23,5 +31,5 @@
     </link>
     <gazebo reference="laser_frame">
-        <material>Gazebo/Red</material>
+        <material>Gazebo/Black</material>
         <sensor name="laser" type="ray">
             <pose> 0 0 0 0 0 0 </pose>
@@ -37,5 +45,5 @@
                 </scan>
                 <range>
-                    <min>0.1</min>
+                    <min>0.25</min>
                     <max>12</max>
                 </range>
@@ -50,3 +58,21 @@
         </sensor>
     </gazebo>
+    <!-- Ground truth pose -->
+    <gazebo>
+      <plugin name="groud_truth_pose" filename="libgazebo_ros_p3d.so">
+        <always_on>true</always_on>
+        <update_rate>50.0</update_rate>
+        <body_name>base_link</body_name>
+        <topic_name>odom</topic_name>
+        <gaussian_noise>0.00</gaussian_noise>
+        <frame_name>world</frame_name>
+        <tf_frame_name>world</tf_frame_name>
+        <tf_prefix>odom_groud_truth_pose</tf_prefix>
+        <xyz_offset>0 0 0</xyz_offset>
+        <rpy_offset>0 0 0</rpy_offset>
+        <ros>
+            <remapping>/odom:=odom_groud_truth_pose</remapping>
+        </ros>
+      </plugin>
+    </gazebo>
 </robot>
