Commit message: update

File: zhbbot/src/zhbbot_description/description/zhbbot_core.xacro (robot description, xacro)
@@ -6,4 +6,12 @@
     <!-- BASE LINK -->
     <link name="base_link">
+        <visual>
+        <geometry>
+            <box size="0.01 0.01 0.01"/>
+        </geometry>
+        <material name="Cyan">
+            <color rgba="0 1.0 1.0 1.0"/>
+        </material>
+        </visual>
     </link>
     <!-- BASE_FOOTPRINT LINK -->
@@ -11,5 +19,5 @@
         <parent link="base_link"/>
         <child link="base_footprint"/>
-        <origin xyz="0 0 0" rpy="0 0 0"/>
+        <origin xyz="0 0 ${-wheel_radius + wheel_offset_z}" rpy="0 0 0"/>
     </joint>
     <link name="base_footprint">

Commit message: Done Cal Score Trajectory

File: zhbbot/src/zhbbot_description/description/zhbbot_core.xacro (robot description, xacro)
@@ -16,10 +16,17 @@
     </link>
     <!-- BASE_FOOTPRINT LINK -->
-    <joint name="base_footprint_joint" type="fixed">
+    <!-- For Velocity Controller -->
+    <!-- <joint name="base_footprint_joint" type="fixed">
         <parent link="base_footprint"/>
         <child link="base_link"/>
-        <!-- <origin xyz="0 0 ${-wheel_radius + wheel_offset_z}" rpy="0 0 0"/> -->
         <origin xyz="0 0 0" rpy="0 0 0"/>
-    </joint>
+    </joint> -->
+    <!-- For Differantial Drive Controller -->
+    <joint name="base_footprint_joint" type="fixed">
+        <parent link="base_link"/>
+        <child link="base_footprint"/>
+        <origin xyz="0 0 0" rpy="0 0 0"/>
+    </joint>
+    <!-- <origin xyz="0 0 ${-wheel_radius + wheel_offset_z}" rpy="0 0 0"/> -->
     <link name="base_footprint">
     </link>

Commit message: update

File: zhbbot/src/zhbbot_description/description/zhbbot_core.xacro (robot description, xacro)
@@ -17,15 +17,15 @@
     <!-- BASE_FOOTPRINT LINK -->
     <!-- For Velocity Controller -->
-    <!-- <joint name="base_footprint_joint" type="fixed">
+    <joint name="base_footprint_joint" type="fixed">
         <parent link="base_footprint"/>
         <child link="base_link"/>
         <origin xyz="0 0 0" rpy="0 0 0"/>
-    </joint> -->
+    </joint>
     <!-- For Differantial Drive Controller -->
-    <joint name="base_footprint_joint" type="fixed">
+    <!-- <joint name="base_footprint_joint" type="fixed">
         <parent link="base_link"/>
         <child link="base_footprint"/>
         <origin xyz="0 0 0" rpy="0 0 0"/>
-    </joint>
+    </joint> -->
     <!-- <origin xyz="0 0 ${-wheel_radius + wheel_offset_z}" rpy="0 0 0"/> -->
     <link name="base_footprint">
