Commit message: update

File: zhbbot/src/zhbbot_description/description/zhbbot_addon.xacro (robot description, xacro)
@@ -63,5 +63,5 @@
         <always_on>true</always_on>
         <update_rate>50.0</update_rate>
-        <body_name>base_link</body_name>
+        <body_name>base_footprint</body_name>
         <topic_name>odom</topic_name>
         <gaussian_noise>0.00</gaussian_noise>

File: zhbbot/src/zhbbot_description/description/zhbbot_core.xacro (robot description, xacro)
@@ -17,7 +17,8 @@
     <!-- BASE_FOOTPRINT LINK -->
     <joint name="base_footprint_joint" type="fixed">
-        <parent link="base_link"/>
-        <child link="base_footprint"/>
-        <origin xyz="0 0 ${-wheel_radius + wheel_offset_z}" rpy="0 0 0"/>
+        <parent link="base_footprint"/>
+        <child link="base_link"/>
+        <!-- <origin xyz="0 0 ${-wheel_radius + wheel_offset_z}" rpy="0 0 0"/> -->
+        <origin xyz="0 0 0" rpy="0 0 0"/>
     </joint>
     <link name="base_footprint">

Commit message: update

File: zhbbot/src/zhbbot_description/description/zhbbot_addon.xacro (robot description, xacro)
@@ -1,58 +1,38 @@
 <?xml version="1.0"?>
 <robot xmlns:xacro="http://www.ros.org/wiki/xacro" >
-    <!-- Laser  -->
-    <joint name="laser_joint" type="fixed">
-        <parent link="base_link"/>
-        <child link="laser_frame"/>
-        <origin xyz="0.122 0 0.312" rpy="0 0 0"/>
-    </joint>
-    <link name="laser_frame">
-        <visual>
-            <geometry>
-                <cylinder radius="0.05" length="0.04"/>
-            </geometry>
-            <material name="red"/>
-        </visual>
-        <visual>
-            <origin xyz="0 0 -0.05"/>
-            <geometry>
-                <cylinder radius="0.01" length="0.1"/>
-            </geometry>
-            <material name="red"/>
-        </visual>
-        <collision>
-            <geometry>
-                <cylinder radius="0.05" length="0.04"/>
-            </geometry>
-        </collision>
-        <xacro:inertial_cylinder mass="0.1" length="0.04" radius="0.05">
-            <origin xyz="0 0 0" rpy="0 0 0"/>
-        </xacro:inertial_cylinder>
-    </link>
-    <gazebo reference="laser_frame">
-        <material>Gazebo/Black</material>
-        <sensor name="lidar_sensor" type="ray">
-            <pose> 0 0 0 0 0 0 </pose>
+    <gazebo reference="lidar_link">
+        <sensor type="ray" name="lidar_sensor">
+            <pose>0 0 0 0 0 0</pose>
             <visualize>true</visualize>
-            <update_rate>10</update_rate>
+            <always_on>true</always_on>
+            <update_rate>40</update_rate>
             <ray>
                 <scan>
                     <horizontal>
-                        <samples>360</samples>
-                        <min_angle>-3.14</min_angle>
-                        <max_angle>3.14</max_angle>
+                        <samples>720</samples>
+                        <resolution>1</resolution>
+                        <min_angle>-3.1415926</min_angle>
+                        <max_angle>3.1415926</max_angle>
                     </horizontal>
                 </scan>
                 <range>
-                    <min>0.25</min>
-                    <max>20</max>
+                    <min>0.05</min>
+                    <max>16.0</max>
+                    <resolution>0.03</resolution>
                 </range>
+                <noise>
+                    <type>gaussian</type>
+                    <mean>0.0</mean>
+                    <stddev>0.03</stddev>
+                </noise>
             </ray>
-            <plugin name="laser_controller" filename="libgazebo_ros_ray_sensor.so">
+            <plugin name="lidar_controller" filename="libgazebo_ros_ray_sensor.so">
                 <ros>
-                    <argument>~/out:=scan</argument>
+                    <remapping>~/out:=scan</remapping>
                 </ros>
                 <output_type>sensor_msgs/LaserScan</output_type>
-                <frame_name>laser_frame</frame_name>
+                <topicName>scan</topicName>
+                <frame_name>lidar_link</frame_name>
+                <frame_Id>lidar_link</frame_Id>
             </plugin>
         </sensor>

File: zhbbot/src/zhbbot_description/description/zhbbot_core.xacro (robot description, xacro)
@@ -225,3 +225,32 @@
         <mu2 value="0.001"/>
     </gazebo>
+    <!-- Laser  -->
+    <joint name="laser_joint" type="fixed">
+        <parent link="base_link"/>
+        <child link="lidar_link"/>
+        <origin xyz="0.122 0 0.312" rpy="0 0 0"/>
+    </joint>
+    <link name="lidar_link">
+        <visual>
+            <geometry>
+                <cylinder radius="0.05" length="0.04"/>
+            </geometry>
+            <material name="red"/>
+        </visual>
+        <visual>
+            <origin xyz="0 0 -0.05"/>
+            <geometry>
+                <cylinder radius="0.01" length="0.1"/>
+            </geometry>
+            <material name="red"/>
+        </visual>
+        <collision>
+            <geometry>
+                <cylinder radius="0.05" length="0.04"/>
+            </geometry>
+        </collision>
+        <xacro:inertial_cylinder mass="0.1" length="0.04" radius="0.05">
+            <origin xyz="0 0 0" rpy="0 0 0"/>
+        </xacro:inertial_cylinder>
+    </link>
 </robot>

File: zhbbot/src/zhbbot_description/description/zhbbot_robot.urdf.xacro (robot description, xacro)
@@ -6,5 +6,4 @@
     <xacro:include filename="zhbbot_addon.xacro" />
     <!-- ADD Control -->
-    <!-- <xacro:include filename="gazebo_control.xacro" /> -->
     <xacro:include filename="zhbbot_ros2control.xacro" />
 </robot>
