Commit message: update

File: zhbbot/src/zhbbot_description/description/zhbbot_ros2control.xacro (robot description, xacro)
@@ -1,34 +1,36 @@
 <?xml version="1.0"?>
 <robot xmlns:xacro="http://www.ros.org/wiki/xacro">
-  <!-- ===== Gazebo ROS2_CONTROL plugin ===== -->
-    <gazebo>
-        <plugin filename="libgazebo_ros2_control.so" name="gazebo_ros2_control">
-          <robot_sim_type>gazebo_ros2_control/GazeboSystem</robot_sim_type>
-          <parameters>$(find zhbbot_description)/config/zhbbot_controller.yaml</parameters>
-        </plugin>
-    </gazebo>
-  <!-- ========== ROS2 CONTROL ========== -->
-    <ros2_control name="GazeboSystem" type="system">
-      <hardware>
-          <plugin>gazebo_ros2_control/GazeboSystem</plugin>
-      </hardware>
-      <joint name="left_wheel_joint">
-          <command_interface name="velocity">
-              <param name="min">-10</param>
-              <param name="max">10</param>
-          </command_interface>
-          <state_interface name="velocity"/>
-          <state_interface name="position"/>
-          <state_interface name="effort"/>
-      </joint>
-      <joint name="right_wheel_joint">
-          <command_interface name="velocity">
-              <param name="min">-10</param>
-              <param name="max">10</param>
-          </command_interface>
-          <state_interface name="velocity"/>
-          <state_interface name="position"/>
-          <state_interface name="effort"/>
-      </joint>
-    </ros2_control>
+  <xacro:macro name="zhbbot_control" params="">
+    <!-- ===== Gazebo ROS2_CONTROL plugin ===== -->
+      <gazebo>
+          <plugin filename="libgazebo_ros2_control.so" name="gazebo_ros2_control">
+            <robot_sim_type>gazebo_ros2_control/GazeboSystem</robot_sim_type>
+            <parameters>$(find zhbbot_description)/config/zhbbot_controller.yaml</parameters>
+          </plugin>
+      </gazebo>
+    <!-- ========== ROS2 CONTROL ========== -->
+      <ros2_control name="GazeboSystem" type="system">
+        <hardware>
+            <plugin>gazebo_ros2_control/GazeboSystem</plugin>
+        </hardware>
+        <joint name="left_wheel_joint">
+            <command_interface name="velocity">
+                <param name="min">-10</param>
+                <param name="max">10</param>
+            </command_interface>
+            <state_interface name="velocity"/>
+            <state_interface name="position"/>
+            <state_interface name="effort"/>
+        </joint>
+        <joint name="right_wheel_joint">
+            <command_interface name="velocity">
+                <param name="min">-10</param>
+                <param name="max">10</param>
+            </command_interface>
+            <state_interface name="velocity"/>
+            <state_interface name="position"/>
+            <state_interface name="effort"/>
+        </joint>
+      </ros2_control>
+  </xacro:macro>
 </robot>
