Commit message: joy control

File: carverabwu/src/testbot_description/description/testbot_core.urdf.xacro (robot description, xacro)
@@ -20,15 +20,15 @@
         <!-- BASE_FOOTPRINT LINK -->
         <!-- For Velocity Controller -->
-        <joint name="base_footprint_joint" type="fixed">
+        <!-- <joint name="base_footprint_joint" type="fixed">
             <parent link="base_footprint"/>
             <child link="base_link"/>
             <origin xyz="0 0 0" rpy="0 0 0"/>
-        </joint>
+        </joint> -->
         <!-- For Differantial Drive Controller -->
-        <!-- <joint name="base_footprint_joint" type="fixed">
+        <joint name="base_footprint_joint" type="fixed">
             <parent link="base_link"/>
             <child link="base_footprint"/>
             <origin xyz="0 0 0" rpy="0 0 0"/>
-        </joint> -->
+        </joint>
         <!-- <origin xyz="0 0 ${-wheel_radius + wheel_offset_z}" rpy="0 0 0"/> -->
         <link name="base_footprint">

File: carverabwu/src/testbot_description/description/testbot_ros2control.xacro (robot description, xacro)
@@ -48,5 +48,5 @@
               <plugin name="laser_controller" filename="libgazebo_ros_ray_sensor.so">
                   <ros>
-                      <argument>~/out:=scan</argument>
+                      <argument>--remap ~/out:=scan</argument>
                   </ros>
                   <output_type>sensor_msgs/LaserScan</output_type>
