Commit message: update

File: carverabwu/src/testbot_description/description/testbot.urdf.xacro (robot description, xacro)
@@ -3,3 +3,5 @@
     <xacro:include filename="testbot_core.urdf.xacro" />
     <xacro:testbot_core/>
+    <xacro:include filename="sensor_lidar.xacro" />
+    <xacro:include filename="sensor_depth_camera.xacro" />
 </robot>

File: carverabwu/src/testbot_description/description/testbot_core.urdf.xacro (robot description, xacro)
@@ -228,28 +228,4 @@
             <mu2 value="0.001"/>
         </gazebo>
-        <!-- Laser  -->
-        <joint name="laser_joint" type="fixed">
-            <parent link="base_link"/>
-            <child link="lidar_link"/>
-            <origin xyz="0.122 0 0.312" rpy="0 0 0"/>
-        </joint>
-        <link name="lidar_link">
-            <visual>
-                <geometry>
-                    <cylinder radius="0.05" length="0.04"/>
-                </geometry>
-                <material name="red"/>
-            </visual>
-            <visual>
-                <origin xyz="0 0 -0.05"/>
-                <geometry>
-                    <cylinder radius="0.01" length="0.1"/>
-                </geometry>
-                <material name="red"/>
-            </visual>
-        </link>
-        <gazebo reference="lidar_link">
-                <material>Gazebo/Red</material>
-        </gazebo>
     </xacro:macro>
 </robot>

File: carverabwu/src/testbot_description/description/testbot_ros2control.xacro (robot description, xacro)
@@ -27,32 +27,4 @@
           </plugin>
       </gazebo>
-    <!-- Laser sensor -->
-      <gazebo reference="lidar_link">
-          <sensor name="laser" type="ray">
-              <pose> 0 0 0 0 0 0 </pose>
-              <visualize>true</visualize>
-              <update_rate>5</update_rate>
-              <ray>
-                  <scan>
-                      <horizontal>
-                          <samples>360</samples>
-                          <min_angle>-3.14</min_angle>
-                          <max_angle>3.14</max_angle>
-                      </horizontal>
-                  </scan>
-                  <range>
-                      <min>0.25</min>
-                      <max>20</max>
-                  </range>
-              </ray>
-              <plugin name="laser_controller" filename="libgazebo_ros_ray_sensor.so">
-                  <ros>
-                      <argument>--remap ~/out:=scan</argument>
-                  </ros>
-                  <output_type>sensor_msgs/LaserScan</output_type>
-                  <frame_name>lidar_link</frame_name>
-              </plugin>
-          </sensor>
-      </gazebo>
     <!-- ========== ROS2 CONTROL ========== -->
       <ros2_control name="GazeboSystem" type="system">
