Commit message: update

File: carverabwu/src/testbot_description/description/camera.xacro (robot description, xacro)
@@ -11,5 +11,12 @@
                 <box size="0.010 0.03 0.03"/>
             </geometry>
-            <material name="red"/>
+            <material name="black"/>
+        </visual>
+        <visual>
+            <origin xyz="0 0 -0.05"/>
+            <geometry>
+                <cylinder radius="0.002" length="0.1"/>
+            </geometry>
+            <material name="black"/>
         </visual>
     </link>
@@ -22,24 +29,22 @@
     <gazebo reference="camera_link">
         <material>Gazebo/Black</material>
-        <sensor name="camera" type="depth">
+        <sensor name="camera" type="camera">
             <pose> 0 0 0 0 0 0 </pose>
             <visualize>true</visualize>
-            <update_rate>30</update_rate>
+            <update_rate>10</update_rate>
             <camera>
                 <horizontal_fov>1.089</horizontal_fov>
                 <image>
-                    <format>B8G8R8</format>
-                    <width>1280</width>
-                    <height>720</height>
+                    <format>R8G8B8</format>
+                    <width>640</width>
+                    <height>480</height>
                 </image>
                 <clip>
                     <near>0.05</near>
-                    <far>6.0</far>
+                    <far>8.0</far>
                 </clip>
             </camera>
             <plugin name="camera_controller" filename="libgazebo_ros_camera.so">
                 <frame_name>camera_link_optical</frame_name>
-                <min_depth>0.1</min_depth>
-                <max_depth>6.0</max_depth>
             </plugin>
         </sensor>

File: carverabwu/src/testbot_description/description/testbot.urdf.xacro (robot description, xacro)
@@ -5,3 +5,4 @@
     <xacro:include filename="sensor_lidar.xacro" />
     <xacro:include filename="sensor_depth_camera.xacro" />
+    <!-- <xacro:include filename="camera.xacro" /> -->
 </robot>
