Commit message: Update pmzbsavy

File: pmzbsavy/src/pmzbsavy_description/description/pmzbsavy.urdf.xacro (robot description, xacro)
@@ -1,5 +1,7 @@
 <?xml version="1.0"?>
 <robot xmlns:xacro="http://www.ros.org/wiki/xacro"  name="robot">
-    <xacro:include filename="pmzbsavy_core.urdf.xacro" />
+    <!-- <xacro:include filename="pmzbsavy_core.urdf.xacro" />
+    <xacro:pmzbsavy_core/> -->
+    <xacro:include filename="pmzbsavy_core_perfect.urdf.xacro" />
     <xacro:pmzbsavy_core/>
 </robot>

File: pmzbsavy/src/pmzbsavy_description/description/pmzbsavy_common.xacro (robot description, xacro)
@@ -39,12 +39,12 @@
     <xacro:property name="chassis_height" value="0.138" scope="parent"/>
     <xacro:property name="chassis_mass" value="1.0" scope="parent"/>
-    <xacro:property name="wheel_radius" value="0.075" scope="parent"/>
-    <xacro:property name="wheel_thickness" value="0.026" scope="parent"/>
-    <xacro:property name="wheel_mass" value="50" scope="parent"/>
+    <xacro:property name="wheel_radius" value="0.05" scope="parent"/>
+    <xacro:property name="wheel_thickness" value="0.06" scope="parent"/>
+    <xacro:property name="wheel_mass" value="0.45133" scope="parent"/>
     <xacro:property name="wheel_offset_x" value="0.4" scope="parent"/>
     <xacro:property name="wheel_offset_y" value="0.2" scope="parent"/>
     <xacro:property name="wheel_offset_z" value="0.0001" scope="parent"/>
     <xacro:property name="caster_wheel_radius" value="0.05" scope="parent"/>
-    <xacro:property name="caster_wheel_mass" value="0.01" scope="parent"/>
+    <xacro:property name="caster_wheel_mass" value="0.32379" scope="parent"/>
     <xacro:property name="caster_wheel_offset_x" value="0.3" scope="parent"/>
     <xacro:property name="caster_wheel_offset_y" value="0.2" scope="parent"/>

File: pmzbsavy/src/pmzbsavy_description/description/pmzbsavy_core_perfect.urdf.xacro (robot description, xacro)
@@ -47,18 +47,7 @@
                 </geometry>
             </collision>
-            <inertial>
-                <origin
-                    xyz="0.01046951 0.00650223 0.19582248"
-                    rpy="0 0 0" />
-                <mass
-                    value="38.3" />
-                <inertia
-                    ixx="0.86919058"
-                    ixy="0.03016623"
-                    ixz="-0.00361722"
-                    iyy="1.19587445"
-                    iyz="0.01825918"
-                    izz="1.36842641" />
-            </inertial>
+            <xacro:inertial_box mass="38.3" x="0.516" y="0.4876" z="0.295">
+            <origin xyz="0.0 0.0 0.2335" rpy="0 0 0"/>
+            </xacro:inertial_box>
         </link>
         <!-- LEFT WHEEL -->
@@ -70,31 +59,18 @@
         </joint>
         <link name="left_wheel">
-            <visual>
-                <origin xyz="0 0 0"/>
-                <geometry>
-                    <mesh filename="file://$(find pmzbsavy_description)/meshes/Drivewheel.STL"/>
+        <visual>
+                <geometry>
+                    <cylinder radius="${wheel_radius}" length="${wheel_thickness}"/>
                 </geometry>
                 <material name="blue"/>
             </visual>
             <collision>
-                <origin xyz="0 0 0"/>
-                <geometry>
-                    <mesh filename="file://$(find pmzbsavy_description)/meshes/Drivewheel.STL"/>
-                </geometry>
-            </collision>
-            <inertial>
-                <origin
-                    xyz="0 -2.666E-5 0.03"
-                    rpy="0 0 0" />
-                <mass
-                    value="0.45133" />
-                <inertia
-                    ixx="0.00042932"
-                    ixy="0.0"
-                    ixz="0.0"
-                    iyy="0.00042945"
-                    iyz="0.0"
-                    izz="0.00058797" />
-            </inertial>
+                <geometry>
+                    <sphere radius="${wheel_radius}"/>
+                </geometry>
+            </collision>
+            <xacro:inertial_cylinder mass="${wheel_mass}" length="${wheel_thickness}" radius="${wheel_radius}">
+                <origin xyz="0 0 0" rpy="0 0 0"/>
+            </xacro:inertial_cylinder>
         </link>
         <gazebo reference="left_wheel">
@@ -110,30 +86,17 @@
         <link name="right_wheel">
             <visual>
-                <origin xyz="0 0 0"/>
-                <geometry>
-                    <mesh filename="file://$(find pmzbsavy_description)/meshes/Drivewheel.STL"/>
+                <geometry>
+                    <cylinder radius="${wheel_radius}" length="${wheel_thickness}"/>
                 </geometry>
                 <material name="blue"/>
             </visual>
             <collision>
-                <origin xyz="0 0 0"/>
-                <geometry>
-                    <mesh filename="file://$(find pmzbsavy_description)/meshes/Drivewheel.STL"/>
-                </geometry>
-            </collision>
-            <inertial>
-                <origin
-                    xyz="0 -2.666E-5 0.03"
-                    rpy="0 0 0" />
-                <mass
-                    value="0.45133" />
-                <inertia
-                    ixx="0.00042932"
-                    ixy="0.0"
-                    ixz="0.0"
-                    iyy="0.00042945"
-                    iyz="0.0"
-                    izz="0.00058797" />
-            </inertial>
+                <geometry>
+                    <sphere radius="${wheel_radius}"/>
+                </geometry>
+            </collision>
+            <xacro:inertial_cylinder mass="${wheel_mass}" length="${wheel_thickness}" radius="${wheel_radius}">
+                <origin xyz="0 0 0" rpy="0 0 0"/>
+            </xacro:inertial_cylinder>
         </link>
         <gazebo reference="right_wheel">
@@ -144,34 +107,21 @@
             <parent link="base_link"/>
             <child link="caster_wheel_f_r"/>
-            <origin xyz="0.20490726 -0.135475 0.0824" rpy="0 0 0"/>
+            <origin xyz="0.20490726 -0.135475 0.0001" rpy="0 0 0"/>
         </joint>
         <link name="caster_wheel_f_r">
             <visual>
-                <origin xyz="0 0 0"/>
-                <geometry>
-                    <mesh filename="file://$(find pmzbsavy_description)/meshes/Castor_100.STL"/>
-                </geometry>
-                <material name="white"/>
-            </visual>
-            <collision>
-                <origin xyz="0 0 0"/>
-                <geometry>
-                    <mesh filename="file://$(find pmzbsavy_description)/meshes/Castor_100.STL"/>
-                </geometry>
-            </collision>
-            <inertial>
-                <origin
-                    xyz="-0.03218009 0 -0.07621536"
-                    rpy="0 0 0" />
-                <mass
-                    value="0.32379" />
-                <inertia
-                    ixx="0.00032464"
-                    ixy="0.0"
-                    ixz="6.086E-5"
-                    iyy="0.00047939"
-                    iyz="0.0"
-                    izz="0.00026272" />
-            </inertial>
+                <geometry>
+                    <sphere radius="${caster_wheel_radius}"/>
+                </geometry>
+                <material name="white"/>
+            </visual>
+            <collision>
+                <geometry>
+                    <sphere radius="${caster_wheel_radius}"/>
+                </geometry>
+            </collision>
+            <xacro:inertial_sphere mass="${caster_wheel_mass}" radius="${caster_wheel_radius}">
+                <origin xyz="0 0 0" rpy="0 0 0"/>
+            </xacro:inertial_sphere>
         </link>
         <gazebo reference="caster_wheel_f_r">
@@ -184,34 +134,21 @@
             <parent link="base_link"/>
             <child link="caster_wheel_f_l"/>
-            <origin xyz="0.20490726 0.135475 0.0824" rpy="0 0 0"/>
+            <origin xyz="0.20490726 0.135475 0.0001" rpy="0 0 0"/>
         </joint>
         <link name="caster_wheel_f_l">
             <visual>
-                <origin xyz="0 0 0"/>
-                <geometry>
-                    <mesh filename="file://$(find pmzbsavy_description)/meshes/Castor_100.STL"/>
-                </geometry>
-                <material name="white"/>
-            </visual>
-            <collision>
-                <origin xyz="0 0 0"/>
-                <geometry>
-                    <mesh filename="file://$(find pmzbsavy_description)/meshes/Castor_100.STL"/>
-                </geometry>
-            </collision>
-            <inertial>
-                <origin
-                    xyz="-0.03218009 0 -0.07621536"
-                    rpy="0 0 0" />
-                <mass
-                    value="0.32379" />
-                <inertia
-                    ixx="0.00032464"
-                    ixy="0.0"
-                    ixz="6.086E-5"
-                    iyy="0.00047939"
-                    iyz="0.0"
-                    izz="0.00026272" />
-            </inertial>
+                <geometry>
+                    <sphere radius="${caster_wheel_radius}"/>
+                </geometry>
+                <material name="white"/>
+            </visual>
+            <collision>
+                <geometry>
+                    <sphere radius="${caster_wheel_radius}"/>
+                </geometry>
+            </collision>
+            <xacro:inertial_sphere mass="${caster_wheel_mass}" radius="${caster_wheel_radius}">
+                <origin xyz="0 0 0" rpy="0 0 0"/>
+            </xacro:inertial_sphere>
         </link>
         <gazebo reference="caster_wheel_f_l">
@@ -224,34 +161,21 @@
             <parent link="base_link"/>
             <child link="caster_wheel_r_r"/>
-            <origin xyz="-0.14804637 -0.135525 0.0824" rpy="0 0 0"/>
+            <origin xyz="-0.14804637 -0.135475 0.0001" rpy="0 0 0"/>
         </joint>
         <link name="caster_wheel_r_r">
             <visual>
-                <origin xyz="0 0 0"/>
-                <geometry>
-                    <mesh filename="file://$(find pmzbsavy_description)/meshes/Castor_100.STL"/>
-                </geometry>
-                <material name="white"/>
-            </visual>
-            <collision>
-                <origin xyz="0 0 0"/>
-                <geometry>
-                    <mesh filename="file://$(find pmzbsavy_description)/meshes/Castor_100.STL"/>
-                </geometry>
-            </collision>
-            <inertial>
-                <origin
-                    xyz="-0.03218009 0 -0.07621536"
-                    rpy="0 0 0" />
-                <mass
-                    value="0.32379" />
-                <inertia
-                    ixx="0.00032464"
-                    ixy="0.0"
-                    ixz="6.086E-5"
-                    iyy="0.00047939"
-                    iyz="0.0"
-                    izz="0.00026272" />
-            </inertial>
+                <geometry>
+                    <sphere radius="${caster_wheel_radius}"/>
+                </geometry>
+                <material name="white"/>
+            </visual>
+            <collision>
+                <geometry>
+                    <sphere radius="${caster_wheel_radius}"/>
+                </geometry>
+            </collision>
+            <xacro:inertial_sphere mass="${caster_wheel_mass}" radius="${caster_wheel_radius}">
+                <origin xyz="0 0 0" rpy="0 0 0"/>
+            </xacro:inertial_sphere>
         </link>
         <gazebo reference="caster_wheel_r_r">
@@ -264,34 +188,21 @@
             <parent link="base_link"/>
             <child link="caster_wheel_r_l"/>
-            <origin xyz="-0.14804637 0.135475 0.0824" rpy="0 0 0"/>
+            <origin xyz="-0.14804637 0.135475 0.0001" rpy="0 0 0"/>
         </joint>
         <link name="caster_wheel_r_l">
             <visual>
-                <origin xyz="0 0 0"/>
-                <geometry>
-                    <mesh filename="file://$(find pmzbsavy_description)/meshes/Castor_100.STL"/>
-                </geometry>
-                <material name="white"/>
-            </visual>
-            <collision>
-                <origin xyz="0 0 0"/>
-                <geometry>
-                    <mesh filename="file://$(find pmzbsavy_description)/meshes/Castor_100.STL"/>
-                </geometry>
-            </collision>
-            <inertial>
-                <origin
-                    xyz="-0.03218009 0 -0.07621536"
-                    rpy="0 0 0" />
-                <mass
-                    value="0.32379" />
-                <inertia
-                    ixx="0.00032464"
-                    ixy="0.0"
-                    ixz="6.086E-5"
-                    iyy="0.00047939"
-                    iyz="0.0"
-                    izz="0.00026272" />
-            </inertial>
+                <geometry>
+                    <sphere radius="${caster_wheel_radius}"/>
+                </geometry>
+                <material name="white"/>
+            </visual>
+            <collision>
+                <geometry>
+                    <sphere radius="${caster_wheel_radius}"/>
+                </geometry>
+            </collision>
+            <xacro:inertial_sphere mass="${caster_wheel_mass}" radius="${caster_wheel_radius}">
+                <origin xyz="0 0 0" rpy="0 0 0"/>
+            </xacro:inertial_sphere>
         </link>
         <gazebo reference="caster_wheel_r_l">

File: zhbbot/src/zhbbot_description/description/zhbbot_core.urdf.xacro (robot description, xacro)
@@ -64,7 +64,28 @@
             </geometry>
         </collision>
-        <xacro:inertial_box mass="100" x="${chassis_length}" y="${chassis_width}" z="${chassis_height}">
+        <!-- <xacro:inertial_box mass="100" x="${chassis_length}" y="${chassis_width}" z="${chassis_height}">
             <origin xyz="${chassis_length/2} 0 ${chassis_height/2}" rpy="0 0 0"/>
-        </xacro:inertial_box>
+        </xacro:inertial_box> -->
+        <inertial>
+                <origin
+                    xyz="${chassis_length/2} 0 ${chassis_height/2}"
+                    rpy="0 0 0" />
+                <mass
+                    value="1000" />
+                <inertia
+                    ixx="0.86919058"
+                    ixy="0.03016623"
+                    ixz="-0.00361722"
+                    iyy="1.19587445"
+                    iyz="0.01825918"
+                    izz="1.36842641" />
+                <!-- <inertia
+                    ixx="0.86919058"
+                    ixy="0.0"
+                    ixz="0.0"
+                    iyy="1.19587445"
+                    iyz="0.0"
+                    izz="1.36842641" /> -->
+            </inertial>
         </link>
         <!-- LEFT WHEEL -->
@@ -255,5 +276,5 @@
             <sensor name="laser" type="ray">
                 <pose> 0 0 0 0 0 0 </pose>
-                <visualize>true</visualize>
+                <visualize>false</visualize>
                 <update_rate>5</update_rate>
                 <ray>

Commit message: Update Collision
- Chassis
- Both Wheels

File: pmzbsavy/src/pmzbsavy_description/description/pmzbsavy.urdf.xacro (robot description, xacro)
@@ -1,7 +1,7 @@
 <?xml version="1.0"?>
 <robot xmlns:xacro="http://www.ros.org/wiki/xacro"  name="robot">
-    <!-- <xacro:include filename="pmzbsavy_core.urdf.xacro" />
-    <xacro:pmzbsavy_core/> -->
     <xacro:include filename="pmzbsavy_core_perfect.urdf.xacro" />
     <xacro:pmzbsavy_core/>
+    <!-- <xacro:include filename="pmzbsavy_core_perfect.urdf.xacro" />
+    <xacro:pmzbsavy_core/> -->
 </robot>

File: pmzbsavy/src/pmzbsavy_description/description/pmzbsavy_core.urdf.xacro (robot description, xacro)
@@ -83,4 +83,9 @@
                 </geometry>
             </collision>
+            <!-- <collision>
+                <geometry>
+                    <sphere radius="${wheel_radius}"/>
+                </geometry>
+            </collision> -->
             <inertial>
                 <origin
@@ -122,4 +127,9 @@
                 </geometry>
             </collision>
+            <!-- <collision>
+                <geometry>
+                    <sphere radius="${wheel_radius}"/>
+                </geometry>
+            </collision> -->
             <inertial>
                 <origin

File: pmzbsavy/src/pmzbsavy_description/description/pmzbsavy_core_perfect.urdf.xacro (robot description, xacro)
@@ -42,7 +42,7 @@
             </visual>
             <collision>
-                <origin xyz="0 0 0"/>
-                <geometry>
-                    <mesh filename="file://$(find pmzbsavy_description)/meshes/URDF_SAVVY.STL"/>
+                <origin xyz="0.03595 -0.00002 0.2385"/>
+                <geometry>
+                    <box size="0.558 0.4876 0.295"/>
                 </geometry>
             </collision>
@@ -55,5 +55,5 @@
             <parent link="base_link"/>
             <child link="left_wheel"/>
-            <origin xyz="0 0.105525 0" rpy="-${pi/2} 0 0" />
+            <origin xyz="0 ${(wheel_thickness/2) + 0.105525} 0" rpy="-${pi/2} 0 0" />
             <axis xyz="0 0 1"/>
         </joint>
@@ -81,5 +81,5 @@
             <parent link="base_link"/>
             <child link="right_wheel"/>
-            <origin xyz="0 -0.105525 0" rpy="${pi/2} 0 0" />
+            <origin xyz="0 -${(wheel_thickness/2) + 0.105525} 0" rpy="${pi/2} 0 0" />
             <axis xyz="0 0 -1"/>
         </joint>
