Commit message: Update Lidar

File: carverabwu/install/carversavvy_description/share/carversavvy_description/description/carversavvy.urdf.xacro (robot description, xacro)
@@ -1 +1 @@
-/home/athimeta/CARVER-Savvy/carverabwu/src/carversavvy_description/description/carversavvy.urdf.xacro
+/home/nuc11/CARVER-Savvy/carverabwu/src/carversavvy_description/description/carversavvy.urdf.xacro

File: carverabwu/install/carversavvy_description/share/carversavvy_description/description/carversavvy_common.xacro (robot description, xacro)
@@ -1 +1 @@
-/home/athimeta/CARVER-Savvy/carverabwu/src/carversavvy_description/description/carversavvy_common.xacro
+/home/nuc11/CARVER-Savvy/carverabwu/src/carversavvy_description/description/carversavvy_common.xacro

File: carverabwu/install/carversavvy_description/share/carversavvy_description/description/carversavvy_core.urdf.xacro (robot description, xacro)
@@ -1 +1 @@
-/home/athimeta/CARVER-Savvy/carverabwu/src/carversavvy_description/description/carversavvy_core.urdf.xacro
+/home/nuc11/CARVER-Savvy/carverabwu/src/carversavvy_description/description/carversavvy_core.urdf.xacro

File: carverabwu/install/carversavvy_description/share/carversavvy_description/description/carversavvy_core_perfect.urdf.xacro (robot description, xacro)
@@ -1 +1 @@
-/home/athimeta/CARVER-Savvy/carverabwu/src/carversavvy_description/description/carversavvy_core_perfect.urdf.xacro
+/home/nuc11/CARVER-Savvy/carverabwu/src/carversavvy_description/description/carversavvy_core_perfect.urdf.xacro

File: carverabwu/install/carversavvy_description/share/carversavvy_description/description/carversavvy_depth_camera.xacro (robot description, xacro)
@@ -1 +1 @@
-/home/athimeta/CARVER-Savvy/carverabwu/src/carversavvy_description/description/carversavvy_depth_camera.xacro
+/home/nuc11/CARVER-Savvy/carverabwu/src/carversavvy_description/description/carversavvy_depth_camera.xacro

File: carverabwu/install/carversavvy_description/share/carversavvy_description/description/carversavvy_lidar.xacro (robot description, xacro)
@@ -1 +1 @@
-/home/athimeta/CARVER-Savvy/carverabwu/src/carversavvy_description/description/carversavvy_lidar.xacro
+/home/nuc11/CARVER-Savvy/carverabwu/src/carversavvy_description/description/carversavvy_lidar.xacro

File: carverabwu/install/carversavvy_description/share/carversavvy_description/description/carversavvy_ros2control.xacro (robot description, xacro)
@@ -1 +1 @@
-/home/athimeta/CARVER-Savvy/carverabwu/src/carversavvy_description/description/carversavvy_ros2control.xacro
+/home/nuc11/CARVER-Savvy/carverabwu/src/carversavvy_description/description/carversavvy_ros2control.xacro

File: carverabwu/install/testbot_description/share/testbot_description/description/camera.xacro (robot description, xacro)
@@ -1 +1 @@
-/home/athimeta/CARVER-Savvy/carverabwu/src/testbot_description/description/camera.xacro
+/home/nuc11/CARVER-Savvy/carverabwu/src/testbot_description/description/camera.xacro

File: carverabwu/install/testbot_description/share/testbot_description/description/inertial_macros.xacro (robot description, xacro)
@@ -1 +1 @@
-/home/athimeta/CARVER-Savvy/carverabwu/src/testbot_description/description/inertial_macros.xacro
+/home/nuc11/CARVER-Savvy/carverabwu/src/testbot_description/description/inertial_macros.xacro

File: carverabwu/install/testbot_description/share/testbot_description/description/sensor_depth_camera.xacro (robot description, xacro)
@@ -1 +1 @@
-/home/athimeta/CARVER-Savvy/carverabwu/src/testbot_description/description/sensor_depth_camera.xacro
+/home/nuc11/CARVER-Savvy/carverabwu/src/testbot_description/description/sensor_depth_camera.xacro

File: carverabwu/install/testbot_description/share/testbot_description/description/sensor_lidar.xacro (robot description, xacro)
@@ -1 +1 @@
-/home/athimeta/CARVER-Savvy/carverabwu/src/testbot_description/description/sensor_lidar.xacro
+/home/nuc11/CARVER-Savvy/carverabwu/src/testbot_description/description/sensor_lidar.xacro

File: carverabwu/install/testbot_description/share/testbot_description/description/testbot.urdf.xacro (robot description, xacro)
@@ -1 +1 @@
-/home/athimeta/CARVER-Savvy/carverabwu/src/testbot_description/description/testbot.urdf.xacro
+/home/nuc11/CARVER-Savvy/carverabwu/src/testbot_description/description/testbot.urdf.xacro

File: carverabwu/install/testbot_description/share/testbot_description/description/testbot_common.xacro (robot description, xacro)
@@ -1 +1 @@
-/home/athimeta/CARVER-Savvy/carverabwu/src/testbot_description/description/testbot_common.xacro
+/home/nuc11/CARVER-Savvy/carverabwu/src/testbot_description/description/testbot_common.xacro

File: carverabwu/install/testbot_description/share/testbot_description/description/testbot_core.urdf.xacro (robot description, xacro)
@@ -1 +1 @@
-/home/athimeta/CARVER-Savvy/carverabwu/src/testbot_description/description/testbot_core.urdf.xacro
+/home/nuc11/CARVER-Savvy/carverabwu/src/testbot_description/description/testbot_core.urdf.xacro

File: carverabwu/install/testbot_description/share/testbot_description/description/testbot_ros2control.xacro (robot description, xacro)
@@ -1 +1 @@
-/home/athimeta/CARVER-Savvy/carverabwu/src/testbot_description/description/testbot_ros2control.xacro
+/home/nuc11/CARVER-Savvy/carverabwu/src/testbot_description/description/testbot_ros2control.xacro

File: carverabwu/src/carversavvy_description/description/carversavvy_lidar.xacro (robot description, xacro)
@@ -5,17 +5,11 @@
         <parent link="base_link"/>
         <child link="lidar_link"/>
-        <origin xyz="0.122 0 0.412" rpy="0 0 0"/>
+        <origin xyz="0.23795 0 0.43660" rpy="0 0 0"/>
     </joint>
     <link name="lidar_link">
         <visual>
+            <origin xyz="0 0 0"/>
             <geometry>
                 <cylinder radius="0.05" length="0.04"/>
-            </geometry>
-            <material name="red"/>
-        </visual>
-        <visual>
-            <origin xyz="0 0 -0.05"/>
-            <geometry>
-                <cylinder radius="0.01" length="0.1"/>
             </geometry>
             <material name="red"/>
