Commit message: update

File: carverabwu/src/awbu_drl/obstacles/cylinder_obstacle_2.urdf (robot description, URDF)
Before this commit: robot cylinder_obstacle_2, 2 links, 1 joints
Links:
- link base_link: geometry collision sphere radius=0.5; visual sphere radius=0.5

File: carverabwu/src/awbu_drl/obstacles/cylinder_obstacle_3.urdf (robot description, URDF)
Before this commit: robot cylinder_obstacle_3, 2 links, 1 joints
Links:
- link base_link: geometry collision sphere radius=0.5; visual sphere radius=0.5

File: carverabwu/src/awbu_drl/obstacles/cylinder_obstacle_4.urdf (robot description, URDF)
Before this commit: robot cylinder_obstacle_4, 2 links, 1 joints
Links:
- link base_link: geometry collision sphere radius=0.5; visual sphere radius=0.5
