Commit message: update and edit lidar

File: carverabwu/src/awbu_drl/obstacles/obstacle_bot.urdf.xacro (robot description, xacro)
@@ -2,4 +2,11 @@
 <robot xmlns:xacro="http://www.ros.org/wiki/xacro" name="obstacle_bot">
     <xacro:include filename="inertial_macros.xacro"/>
+    <xacro:macro name="obstacle_bot_common">
+        <xacro:property name="chassis_length" value="1.0" scope="parent"/>
+        <xacro:property name="chassis_radius" value="0.5" scope="parent"/>
+        <xacro:property name="chassis_mass" value="10" scope="parent"/>
+        <xacro:property name="wheel_radius" value="0.1" scope="parent"/>
+    </xacro:macro>
+    <xacro:obstacle_bot_common/>
     <!-- BASE LINK -->
     <link name="base_link">
@@ -9,25 +16,77 @@
         <parent link="base_link"/>
         <child link="chassis"/>
-        <origin xyz="-0.1 0 0"/>
+        <origin xyz="0 0 ${wheel_radius}" rpy="0 0 0"/>
     </joint>
     <link name="chassis">
         <visual>
-            <origin xyz="0.15 0 0.075"/>
+            <origin xyz="0 0 ${chassis_length/2}"/>
             <geometry>
-                <box size="0.3 0.3 0.15"/>
+                <cylinder radius="${chassis_radius}" length="${chassis_length}"/>
             </geometry>
         </visual>
         <collision>
-            <origin xyz="0.15 0 0.075"/>
+            <origin xyz="0 0 ${chassis_length/2}"/>
             <geometry>
-                <box size="0.3 0.3 0.15"/>
+                <cylinder radius="${chassis_radius}" length="${chassis_length}"/>
             </geometry>
         </collision>
-        <xacro:inertial_box mass="0.5" x="0.3" y="0.3" z="0.15">
-            <origin xyz="0.15 0 0.075" rpy="0 0 0"/>
-        </xacro:inertial_box>
+        <xacro:inertial_cylinder mass="${chassis_mass}" length="${chassis_length}" radius="${chassis_radius}">
+            <origin xyz="0 0 ${chassis_length/2}" rpy="0 0 0"/>
+        </xacro:inertial_cylinder>
     </link>
     <gazebo reference="chassis">
-        <material>Gazebo/White</material>
+        <material>Gazebo/Red</material>
+    </gazebo>
+    <!-- CASTER WHEEL FONT LINK -->
+    <joint name="caster_wheel_font_joint" type="fixed">
+        <parent link="base_link"/>
+        <child link="caster_wheel_font"/>
+        <origin xyz="${chassis_radius - wheel_radius} 0 0" rpy="0 0 0" />
+    </joint>
+    <link name="caster_wheel_font">
+        <visual>
+            <geometry>
+                <sphere radius="${wheel_radius}"/>
+            </geometry>
+        </visual>
+        <collision>
+            <geometry>
+                <sphere radius="${wheel_radius}"/>
+            </geometry>
+        </collision>
+        <xacro:inertial_sphere mass="0.1" radius="${wheel_radius}">
+            <origin xyz="0 0 0" rpy="0 0 0"/>
+        </xacro:inertial_sphere>
+    </link>
+    <gazebo reference="caster_wheel_font">
+        <material>Gazebo/Black</material>
+        <mu1 value="0.001"/>
+        <mu2 value="0.001"/>
+    </gazebo>
+    <!-- CASTER WHEEL BACK LINK -->
+    <joint name="caster_wheel_back_joint" type="fixed">
+        <parent link="base_link"/>
+        <child link="caster_wheel_back"/>
+        <origin xyz="-${chassis_radius - wheel_radius} 0 0" rpy="0 0 0" />
+    </joint>
+    <link name="caster_wheel_back">
+        <visual>
+            <geometry>
+                <sphere radius="${wheel_radius}"/>
+            </geometry>
+        </visual>
+        <collision>
+            <geometry>
+                <sphere radius="${wheel_radius}"/>
+            </geometry>
+        </collision>
+        <xacro:inertial_sphere mass="0.1" radius="${wheel_radius}">
+            <origin xyz="0 0 0" rpy="0 0 0"/>
+        </xacro:inertial_sphere>
+    </link>
+    <gazebo reference="caster_wheel_back">
+        <material>Gazebo/Black</material>
+        <mu1 value="0.001"/>
+        <mu2 value="0.001"/>
     </gazebo>
     <!-- LEFT WHEEL LINK -->
@@ -35,5 +94,5 @@
         <parent link="base_link"/>
         <child link="left_wheel"/>
-        <origin xyz="0 0.175 0" rpy="-${pi/2} 0 0" />
+        <origin xyz="0 ${chassis_radius - wheel_radius} 0" rpy="-${pi/2} 0 0" />
         <axis xyz="0 0 1"/>
     </joint>
@@ -41,15 +100,15 @@
         <visual>
             <geometry>
-                <cylinder radius="0.05" length="0.04"/>
+                <sphere radius="${wheel_radius}"/>
             </geometry>
         </visual>
         <collision>
             <geometry>
-                <cylinder radius="0.05" length="0.04"/>
+                <sphere radius="${wheel_radius}"/>
             </geometry>
         </collision>
-        <xacro:inertial_cylinder mass="0.1" length="0.04" radius="0.05">
+        <xacro:inertial_sphere mass="0.1" radius="${wheel_radius}">
             <origin xyz="0 0 0" rpy="0 0 0"/>
-        </xacro:inertial_cylinder>
+        </xacro:inertial_sphere>
     </link>
     <gazebo reference="left_wheel">
@@ -60,5 +119,5 @@
         <parent link="base_link"/>
         <child link="right_wheel"/>
-        <origin xyz="0 -0.175 0" rpy="${pi/2} 0 0" />
+        <origin xyz="0 -${chassis_radius - wheel_radius} 0" rpy="${pi/2} 0 0" />
         <axis xyz="0 0 -1"/>
     </joint>
@@ -66,44 +125,18 @@
         <visual>
             <geometry>
-                <cylinder radius="0.05" length="0.04"/>
+                <sphere radius="${wheel_radius}"/>
             </geometry>
         </visual>
         <collision>
             <geometry>
-                <cylinder radius="0.05" length="0.04"/>
+                <sphere radius="${wheel_radius}"/>
             </geometry>
         </collision>
-        <xacro:inertial_cylinder mass="0.1" length="0.04" radius="0.05">
+        <xacro:inertial_sphere mass="0.1" radius="${wheel_radius}">
             <origin xyz="0 0 0" rpy="0 0 0"/>
-        </xacro:inertial_cylinder>
+        </xacro:inertial_sphere>
     </link>
     <gazebo reference="right_wheel">
         <material>Gazebo/Blue</material>
-    </gazebo>
-    <!-- CASTER WHEEL LINK -->
-    <joint name="caster_wheel_joint" type="fixed">
-        <parent link="chassis"/>
-        <child link="caster_wheel"/>
-        <origin xyz="0.24 0 0"/>
-    </joint>
-    <link name="caster_wheel">
-        <visual>
-            <geometry>
-                <sphere radius="0.05"/>
-            </geometry>
-        </visual>
-        <collision>
-            <geometry>
-                <sphere radius="0.05"/>
-            </geometry>
-        </collision>
-        <xacro:inertial_sphere mass="0.1" radius="0.05">
-            <origin xyz="0 0 0" rpy="0 0 0"/>
-        </xacro:inertial_sphere>
-    </link>
-    <gazebo reference="caster_wheel">
-        <material>Gazebo/Black</material>
-        <mu1 value="0.001"/>
-        <mu2 value="0.001"/>
     </gazebo>
     <gazebo>
@@ -112,6 +145,6 @@
             <left_joint>left_wheel_joint</left_joint>
             <right_joint>right_wheel_joint</right_joint>
-            <wheel_separation>0.35</wheel_separation>
-            <wheel_diameter>0.1</wheel_diameter>
+            <wheel_separation>${chassis_length}</wheel_separation>
+            <wheel_diameter>${2*wheel_radius}</wheel_diameter>
             <!-- Limits -->
             <max_wheel_torque>200</max_wheel_torque>

File: carverabwu/src/carversavvy_description/description/carversavvy_lidar.xacro (robot description, xacro)
@@ -28,5 +28,5 @@
                 <scan>
                     <horizontal>
-                        <samples>45</samples>
+                        <samples>90</samples>
                         <min_angle>-3.14</min_angle>
                         <max_angle>3.14</max_angle>
@@ -35,5 +35,5 @@
                 <range>
                     <min>0.10</min>
-                    <max>5.0</max>
+                    <max>10.0</max>
                 </range>
             </ray>

Commit message: update stage2

File: carverabwu/src/awbu_drl/obstacles/obstacle_bot.urdf.xacro (robot description, xacro)
@@ -140,4 +140,28 @@
         <material>Gazebo/Blue</material>
     </gazebo>
+    <!-- Font indicator link -->
+    <joint name="font_indicator_joint" type="fixed">
+        <parent link="chassis"/>
+        <child link="font_indicator"/>
+        <origin xyz="${chassis_radius - 0.1} 0 ${chassis_length}" rpy="0 0 0"/>
+    </joint>
+    <link name="font_indicator">
+        <visual>
+            <geometry>
+                <cylinder radius="0.1" length="0.1"/>
+            </geometry>
+        </visual>
+        <collision>
+            <geometry>
+                <cylinder radius="0.1" length="0.1"/>
+            </geometry>
+        </collision>
+        <xacro:inertial_cylinder mass="0.1" length="0.1" radius="0.1">
+            <origin xyz="0 0 0" rpy="0 0 0"/>
+        </xacro:inertial_cylinder>
+    </link>
+    <gazebo reference="font_indicator">
+        <material>Gazebo/Black</material>
+    </gazebo>
     <gazebo>
         <plugin name="diff_drive" filename="libgazebo_ros_diff_drive.so">
@@ -145,5 +169,5 @@
             <left_joint>left_wheel_joint</left_joint>
             <right_joint>right_wheel_joint</right_joint>
-            <wheel_separation>${chassis_length}</wheel_separation>
+            <wheel_separation>${(chassis_radius - wheel_radius)*2}</wheel_separation>
             <wheel_diameter>${2*wheel_radius}</wheel_diameter>
             <!-- Limits -->

File: carverabwu/src/carversavvy_description/description/carversavvy_lidar.xacro (robot description, xacro)
@@ -35,5 +35,5 @@
                 <range>
                     <min>0.07</min>
-                    <max>10.0</max>
+                    <max>12.0</max>
                 </range>
             </ray>

Commit message: update obs size

File: carverabwu/src/awbu_drl/obstacles/obstacle_bot.urdf.xacro (robot description, xacro)
@@ -4,7 +4,7 @@
     <xacro:macro name="obstacle_bot_common">
         <xacro:property name="chassis_length" value="1.0" scope="parent"/>
-        <xacro:property name="chassis_radius" value="0.5" scope="parent"/>
+        <xacro:property name="chassis_radius" value="0.4" scope="parent"/>
         <xacro:property name="chassis_mass" value="10" scope="parent"/>
-        <xacro:property name="wheel_radius" value="0.1" scope="parent"/>
+        <xacro:property name="wheel_radius" value="0.05" scope="parent"/>
     </xacro:macro>
     <xacro:obstacle_bot_common/>
