Commit message: add savvy

File: carverabwu/src/carversavvy_description/description/carversavvy.urdf.xacro (robot description, xacro)
@@ -1,5 +1,5 @@
 <?xml version="1.0"?>
 <robot xmlns:xacro="http://www.ros.org/wiki/xacro"  name="robot">
-    <xacro:include filename="pmzbsavy_core_perfect.urdf.xacro" />
+    <xacro:include filename="carversavvy_core_perfect.urdf.xacro" />
     <xacro:carversavvy_core/>
     <xacro:include filename="carversavvy_ros2control.xacro" />

File: carverabwu/src/carversavvy_description/description/carversavvy_lidar.xacro (robot description, xacro)
@@ -5,5 +5,5 @@
         <parent link="base_link"/>
         <child link="lidar_link"/>
-        <origin xyz="0.122 0 0.312" rpy="0 0 0"/>
+        <origin xyz="0.122 0 0.412" rpy="0 0 0"/>
     </joint>
     <link name="lidar_link">

Commit message: add new description
Co-Authored-By: Athimet Aiewcharoen <71125762+AthimetA@users.noreply.github.com>

File: carverabwu/src/carversavvy_description/description/carversavvy.urdf.xacro (robot description, xacro)
@@ -1,4 +1,4 @@
 <?xml version="1.0"?>
-<robot xmlns:xacro="http://www.ros.org/wiki/xacro"  name="carversavvy">
+<robot xmlns:xacro="http://www.ros.org/wiki/xacro"  name="robot">
     <xacro:include filename="carversavvy_core_perfect.urdf.xacro" />
     <xacro:carversavvy_core/>

File: carverabwu/src/carversavvy_description/description/carversavvy_core_perfect.urdf.xacro (robot description, xacro)
@@ -52,5 +52,5 @@
             <parent link="base_link"/>
             <child link="left_wheel"/>
-            <origin xyz="0 ${(wheel_thickness/2) + 0.105} 0" rpy="-${pi/2} 0 0" />
+            <origin xyz="0 ${(wheel_thickness/2) + 0.105525} 0" rpy="-${pi/2} 0 0" />
             <axis xyz="0 0 1"/>
         </joint>
@@ -78,5 +78,5 @@
             <parent link="base_link"/>
             <child link="right_wheel"/>
-            <origin xyz="0 -${(wheel_thickness/2) + 0.105} 0" rpy="${pi/2} 0 0" />
+            <origin xyz="0 -${(wheel_thickness/2) + 0.105525} 0" rpy="${pi/2} 0 0" />
             <axis xyz="0 0 -1"/>
         </joint>
@@ -104,5 +104,5 @@
             <parent link="base_link"/>
             <child link="caster_wheel_f_r"/>
-            <origin xyz="0.20490726 -0.135475 0.0001" rpy="0 0 0"/>
+            <origin xyz="0.20490726 -0.135475 0.001" rpy="0 0 0"/>
         </joint>
         <link name="caster_wheel_f_r">
@@ -131,5 +131,5 @@
             <parent link="base_link"/>
             <child link="caster_wheel_f_l"/>
-            <origin xyz="0.20490726 0.135475 0.0001" rpy="0 0 0"/>
+            <origin xyz="0.20490726 0.135475 0.001" rpy="0 0 0"/>
         </joint>
         <link name="caster_wheel_f_l">
@@ -158,5 +158,5 @@
             <parent link="base_link"/>
             <child link="caster_wheel_r_r"/>
-            <origin xyz="-0.14804637 -0.135475 0.0001" rpy="0 0 0"/>
+            <origin xyz="-0.14804637 -0.135475 0.001" rpy="0 0 0"/>
         </joint>
         <link name="caster_wheel_r_r">
@@ -185,5 +185,5 @@
             <parent link="base_link"/>
             <child link="caster_wheel_r_l"/>
-            <origin xyz="-0.14804637 0.135475 0.0001" rpy="0 0 0"/>
+            <origin xyz="-0.14804637 0.135475 0.001" rpy="0 0 0"/>
         </joint>
         <link name="caster_wheel_r_l">

File: carverabwu/src/carversavvy_description/description/carversavvy_lidar.xacro (robot description, xacro)
@@ -21,19 +21,19 @@
     <!-- Gazebo Laser sensor -->
     <gazebo reference="lidar_link">
-        <sensor name="laser" type="ray">
+        <sensor name="laser" type="gpu_ray">
             <pose> 0 0 0 0 0 0 </pose>
             <visualize>false</visualize>
-            <update_rate>5</update_rate>
+            <update_rate>50</update_rate>
             <ray>
                 <scan>
                     <horizontal>
-                        <samples>360</samples>
-                        <min_angle>-3.14</min_angle>
-                        <max_angle>3.14</max_angle>
+                        <samples>720</samples>
+                        <min_angle>-3.1415926535</min_angle>
+                        <max_angle>3.1415926535</max_angle>
                     </horizontal>
                 </scan>
                 <range>
-                    <min>0.25</min>
-                    <max>20</max>
+                    <min>0.1</min>
+                    <max>12.0</max>
                 </range>
             </ray>

File: carverabwu/src/carversavvy_description/description/carversavvy_ros2control.xacro (robot description, xacro)
@@ -13,5 +13,5 @@
           <plugin name="groud_truth_pose" filename="libgazebo_ros_p3d.so">
               <always_on>true</always_on>
-              <update_rate>50.0</update_rate>
+              <update_rate>250.0</update_rate>
               <body_name>base_link</body_name>
               <topic_name>odom</topic_name>
@@ -19,9 +19,9 @@
               <frame_name>world</frame_name>
               <tf_frame_name>world</tf_frame_name>
-              <tf_prefix>odom_groud_truth_pose</tf_prefix>
+              <tf_prefix>abwubot_odom_groud_truth_pose</tf_prefix>
               <xyz_offset>0 0 0</xyz_offset>
               <rpy_offset>0 0 0</rpy_offset>
               <ros>
-                  <remapping>/odom:=odom_groud_truth_pose</remapping>
+                  <remapping>/odom:=/abwubot/odom</remapping>
               </ros>
           </plugin>
