Commit message: update

File: carverabwu/src/carversavvy_description/description/carversavvy_core_perfect.urdf.xacro (robot description, xacro)
@@ -104,5 +104,5 @@
             <parent link="base_link"/>
             <child link="caster_wheel_f_r"/>
-            <origin xyz="0.20490726 -0.135475 0.0001" rpy="0 0 0"/>
+            <origin xyz="0.20490726 -0.135475 0.001" rpy="0 0 0"/>
         </joint>
         <link name="caster_wheel_f_r">
@@ -131,5 +131,5 @@
             <parent link="base_link"/>
             <child link="caster_wheel_f_l"/>
-            <origin xyz="0.20490726 0.135475 0.0001" rpy="0 0 0"/>
+            <origin xyz="0.20490726 0.135475 0.001" rpy="0 0 0"/>
         </joint>
         <link name="caster_wheel_f_l">
@@ -158,5 +158,5 @@
             <parent link="base_link"/>
             <child link="caster_wheel_r_r"/>
-            <origin xyz="-0.14804637 -0.135475 0.0001" rpy="0 0 0"/>
+            <origin xyz="-0.14804637 -0.135475 0.001" rpy="0 0 0"/>
         </joint>
         <link name="caster_wheel_r_r">
@@ -185,5 +185,5 @@
             <parent link="base_link"/>
             <child link="caster_wheel_r_l"/>
-            <origin xyz="-0.14804637 0.135475 0.0001" rpy="0 0 0"/>
+            <origin xyz="-0.14804637 0.135475 0.001" rpy="0 0 0"/>
         </joint>
         <link name="caster_wheel_r_l">

File: carverabwu/src/carversavvy_description/description/carversavvy_ros2control.xacro (robot description, xacro)
@@ -13,5 +13,5 @@
           <plugin name="groud_truth_pose" filename="libgazebo_ros_p3d.so">
               <always_on>true</always_on>
-              <update_rate>50.0</update_rate>
+              <update_rate>250.0</update_rate>
               <body_name>base_link</body_name>
               <topic_name>odom</topic_name>

Commit message: Update

File: carverabwu/src/carversavvy_description/description/carversavvy_core_perfect.urdf.xacro (robot description, xacro)
@@ -52,5 +52,5 @@
             <parent link="base_link"/>
             <child link="left_wheel"/>
-            <origin xyz="0 ${(wheel_thickness/2) + 0.105525} 0" rpy="-${pi/2} 0 0" />
+            <origin xyz="0 ${(wheel_thickness/2) + 0.105} 0" rpy="-${pi/2} 0 0" />
             <axis xyz="0 0 1"/>
         </joint>
@@ -78,5 +78,5 @@
             <parent link="base_link"/>
             <child link="right_wheel"/>
-            <origin xyz="0 -${(wheel_thickness/2) + 0.105525} 0" rpy="${pi/2} 0 0" />
+            <origin xyz="0 -${(wheel_thickness/2) + 0.105} 0" rpy="${pi/2} 0 0" />
             <axis xyz="0 0 -1"/>
         </joint>

Commit message: update

File: carverabwu/src/carversavvy_description/description/carversavvy_core_perfect.urdf.xacro (robot description, xacro)
@@ -104,5 +104,5 @@
             <parent link="base_link"/>
             <child link="caster_wheel_f_r"/>
-            <origin xyz="0.20490726 -0.135475 0.001" rpy="0 0 0"/>
+            <origin xyz="0.20490726 -0.135475 0.0001" rpy="0 0 0"/>
         </joint>
         <link name="caster_wheel_f_r">
@@ -131,5 +131,5 @@
             <parent link="base_link"/>
             <child link="caster_wheel_f_l"/>
-            <origin xyz="0.20490726 0.135475 0.001" rpy="0 0 0"/>
+            <origin xyz="0.20490726 0.135475 0.0001" rpy="0 0 0"/>
         </joint>
         <link name="caster_wheel_f_l">
@@ -158,5 +158,5 @@
             <parent link="base_link"/>
             <child link="caster_wheel_r_r"/>
-            <origin xyz="-0.14804637 -0.135475 0.001" rpy="0 0 0"/>
+            <origin xyz="-0.14804637 -0.135475 0.0001" rpy="0 0 0"/>
         </joint>
         <link name="caster_wheel_r_r">
@@ -185,5 +185,5 @@
             <parent link="base_link"/>
             <child link="caster_wheel_r_l"/>
-            <origin xyz="-0.14804637 0.135475 0.001" rpy="0 0 0"/>
+            <origin xyz="-0.14804637 0.135475 0.0001" rpy="0 0 0"/>
         </joint>
         <link name="caster_wheel_r_l">

File: carverabwu/src/carversavvy_description/description/carversavvy_lidar.xacro (robot description, xacro)
@@ -34,6 +34,6 @@
                 </scan>
                 <range>
-                    <min>0.1</min>
-                    <max>12.0</max>
+                    <min>0.15</min>
+                    <max>8.0</max>
                 </range>
             </ray>
